File: compactmacropad.kicad_pcb (KiCad board)
At the start: 2 copper layers, 97.6 x 66.7 mm, 30 parts, among them SW1 RotaryEncoder_Switch, SW3 RotaryEncoder_Switch, U1 MCU_Seeed_XIAO_RP2040

Commit message: New files
Parts:
- added U2: SN74LV1T34DBV, Package_TO_SOT_SMD:SOT-23-5, F.Cu at (2.08, 1.90)
- D10, D14, D15, D16: footprint LED_SMD:LED_SK6812MINI_PLCC4_3.5x3.5mm_P1.75mm -> kicad-keyboard-parts.pretty-master:MX_SK6812MINI-E_REV; moved to F.Cu
- D11, D12, D13: footprint LED_SMD:LED_SK6812MINI_PLCC4_3.5x3.5mm_P1.75mm -> kicad-keyboard-parts.pretty-master:MX_SK6812MINI-E_REV_Rot; moved to F.Cu
- D17, D18, D19, D20: footprint LED_SMD:LED_SK6812MINI_PLCC4_3.5x3.5mm_P1.75mm -> kicad-keyboard-parts.pretty-master:MX_SK6812MINI-E; moved to F.Cu
- moved D17 16.2 mm to (88.8, 77.5)
- moved D19 14.1 mm to (92.5, 96.5)
- moved D20 7.23 mm to (101.9, 106.0)
- moved D14 4.45 mm to (130.5, 101.2), turned to 0 degrees
- moved D16 4.45 mm to (168.5, 101.2), turned to 0 degrees
- moved D15 4.44 mm to (149.5, 101.2), turned to 0 degrees
- moved D11 4.40 mm to (130.5, 82.2)
- moved D13 4.40 mm to (168.5, 82.2)
- moved D12 4.40 mm to (149.5, 82.2)
- moved D10 4.36 mm to (149.5, 63.2), turned to 0 degrees
- moved D18 3.27 mm to (100.7, 83.4)
- moved D4 2.14 mm to (120.9, 89.6)
- moved D5 2.14 mm to (140.0, 89.6)
- moved D6 2.14 mm to (159.0, 89.6)
- moved D7 2.14 mm to (120.9, 108.7)
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Routing:
- net +5V: track 240.4 -> 307.6 mm
- net GND: track 299.8 -> 284.7 mm, vias 8 -> 4
- net Led input: track 38.1 -> 24.5 mm
- net Net-(D14-DIN): track 34.1 -> 24.4 mm
- net Net-(D10-DIN): track 39.4 -> 31.3 mm, vias 0 -> 2
- net Net-(D19-DOUT): track 18.8 -> 13.8 mm
- net Net-(D17-DOUT): track 12.9 -> 17.6 mm
- net Net-(D11-DIN): track 17.5 -> 14.4 mm
- net Net-(D12-DIN): track 17.5 -> 14.4 mm
- net row_2: track 111.6 -> 114.6 mm
- net Net-(D14-DOUT): track 16.3 -> 14.4 mm
- net Net-(D15-DOUT): track 16.3 -> 14.4 mm
- net Net-(D18-DOUT): track 9.25 -> 10.7 mm
- net col_2: track 132.8 -> 134.2 mm
- net col_1: track 131.3 -> 132.6 mm
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